File: 7/KiCAD/RS232C/FM7-RS232C.sch (KiCad schematic (older format))
At the start: 33 parts, among them CN2 DB9_Male, M10 74LS04, M11 8251A, M12 74LS27, M13 74LS11, M2 74LS38, M3 75188, M4 75189, M5 74LS00, M6 74LS32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

Commit message: Added +5V, GND pads.  Unofficially added JP6.  38400bps was already unofficial.
Parts:
- added JP6: Jumper_NO_Small, Connector_PinHeader_2.54mm:PinHeader_1x02_P2.54mm_Vertical, symbol Device:Jumper_NO_Small
- added TP_5V1, TP_GND1: TestPoint, TestPoint:TestPoint_THTPad_D1.5mm_Drill0.7mm, symbol Connector:TestPoint
Connections:
- net +5V: now also TP_5V1.1
- net GNDPWR: now also TP_GND1.1
- net 19200bps: now reaches JP4.1, M8.13 (CP), M8.6 (Q3)
- net at JP1.2, JP2.2, JP3.2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: now also JP6.2
- net 9600bps: now reaches JP3.1, M8.11 (Q0)
- net 4800bps: now reaches JP2.1, M8.10 (Q1)
- net 2400bps: now reaches JP1.1, M8.9 (Q2)
- net 38400bps: now reaches JP5.1, M8.5 (Q2)
- net 76800bps: now reaches M8.4 (Q1)
- net 76800bps: now also JP6.1
- no-connect marks 11 -> 10
Other:
- note added: "Intel 8251 unofficially supports up to 38400bps.\n76800bps never succeeded.\nNonetheless, there might be a compatible chip\nthat can go up to higher bps."
- note added: "Read if ERW=1 and EE=1"
- note added: "Write if ERW=0 and EE=1"
Changed lines of the file:
@@
 	20350 19600 20350 19700
 Wire Wire Line
-	20350 19700 26100 19700
+	20350 19700 22250 19700
 Wire Wire Line
 	20250 18750 20250 18700
@@
 Connection ~ 17350 18600
 Wire Wire Line
-	17350 18600 26500 18600
+	17350 18600 22250 18600
 Connection ~ 17350 19700
 Wire Wire Line
@@
 NoConn ~ 16600 16350
 NoConn ~ 16600 14750
-NoConn ~ 16600 13800
 NoConn ~ 16600 13700
 NoConn ~ 20750 13550
@@
 Text Notes 13750 10050 0    50   ~ 0
 WFD02=\nAB=00000010 and\n~IOS~=0 (IOS=1) and\nEE=1 and\nEQ=1 and\n~ERW~=1 (ERW=0)\n
+Text Notes 17550 12550 0    50   ~ 0
+Read if ERW=1 and EE=1
+Text Notes 17600 12050 0    50   ~ 0
+Write if ERW=0 and EE=1
+Text Label 16600 13900 0    50   ~ 0
+38400bps
+Text Label 16750 14000 0    50   ~ 0
+19200bps
+Text Label 16650 14450 0    50   ~ 0
+9600bps
+Text Label 16650 14550 0    50   ~ 0
+4800bps
+Text Label 16650 14650 0    50   ~ 0
+2400bps
+$Comp
+L Device:Jumper_NO_Small JP6
+U 1 1 61A0FB63
+P 17300 13800
+F 0 "JP6" H 17300 13893 50  0000 C CNN
+F 1 "Jumper_NO_Small" H 17300 13894 50  0001 C CNN
+F 2 "Connector_PinHeader_2.54mm:PinHeader_1x02_P2.54mm_Vertical" H 17300 13800 50  0001 C CNN
+F 3 "~" H 17300 13800 50  0001 C CNN
+	1    17300 13800
+	1    0    0    -1
+$EndComp
+Wire Wire Line
+	17400 13800 17750 13800
+Wire Wire Line
+	17750 13800 17750 13900
+Connection ~ 17750 13900
+Wire Wire Line
+	17200 13800 16600 13800
+Text Label 16600 13800 0    50   ~ 0
+76800bps
+Text Notes 17500 13700 0    50   ~ 0
+Intel 8251 unofficially supports up to 38400bps.\n76800bps never succeeded.\nNonetheless, there might be a compatible chip\nthat can go up to higher bps.
+$Comp
+L Connector:TestPoint TP_5V1
+U 1 1 61AD1210
+P 22250 18600
+F 0 "TP_5V1" H 22308 18718 50  0000 L CNN
+F 1 "TestPoint" H 22308 18627 50  0000 L CNN
+F 2 "TestPoint:TestPoint_THTPad_D1.5mm_Drill0.7mm" H 22450 18600 50  0001 C CNN
+F 3 "~" H 22450 18600 50  0001 C CNN
+	1    22250 18600
+	1    0    0    -1
+$EndComp
+Connection ~ 22250 18600
+Wire Wire Line
+	22250 18600 26500 18600
+$Comp
+L Connector:TestPoint TP_GND1
+U 1 1 61AD166F
+P 22250 19700
+F 0 "TP_GND1" H 22308 19818 50  0000 L CNN
+F 1 "TestPoint" H 22308 19727 50  0000 L CNN
+F 2 "TestPoint:TestPoint_THTPad_D1.5mm_Drill0.7mm" H 22450 19700 50  0001 C CNN
+F 3 "~" H 22450 19700 50  0001 C CNN
+	1    22250 19700
+	1    0    0    -1
+$EndComp
+Connection ~ 22250 19700
+Wire Wire Line
+	22250 19700 26100 19700
 $EndSCHEMATC

Commit message: Optimizing PCB
Other:
- note added: "~ERW"
Changed lines of the file:
@@
 Text Label 9100 10600 0    50   ~ 0
 EE
-Text Label 5850 10500 0    50   ~ 0
+Text Label 9100 10500 0    50   ~ 0
 EQ
 Wire Wire Line
@@
 Text Notes 10300 10100 0    50   ~ 0
 AB1=1
-Text Notes 11300 10150 0    50   ~ 0
-=0\nif AB347=000,AB1=1
 Text Notes 11400 9200 0    50   ~ 0
 =0 if AB02=00
@@
 Wire Wire Line
 	22250 19700 26100 19700
+Text Notes 12400 6700 0    50   ~ 0
+EAB5
+Text Notes 12050 7450 0    50   ~ 0
+EAB1
+Text Notes 12300 6600 0    50   ~ 0
+EAB6
+Text Notes 14250 7000 0    50   ~ 0
+EAB3
+Text Notes 14250 7100 0    50   ~ 0
+EAB4
+Text Notes 14250 7200 0    50   ~ 0
+EAB7
+Text Notes 14100 8000 0    50   ~ 0
+EAB2
+Text Notes 11300 10150 0    50   ~ 0
+=0\nif AB347=000,AB1=1
+Text Notes 10900 10950 0    50   ~ 0
+~ERW
 $EndSCHEMATC
