File: TOWNS/KiCAD/FRAMCard/ICMemCard.kicad_pcb (KiCad board)
At the start: 2 copper layers, 78.5 x 47.2 mm, 19 parts, among them J1 PCMCIA_Connector, Q1 BC846X, Q2 BC846X, U1 FM18W08-SGTR, U2 FM18W08-SGTR, U3 SN74LS32DR

Commit message: Increased re-read count to 16.
Parts:
- added REF**: 2mmX3.5mmPadSMD, PCMCIA:2mmX3.5mmPadSMD, B.Cu at (115.8, 50.7)
- added REF**: 2mmX3.5mmPadSMD, PCMCIA:2mmX3.5mmPadSMD, B.Cu at (115.8, 93.6)
- added REF**: 2mmX3.5mmPadSMD, PCMCIA:2mmX3.5mmPadSMD, B.Cu at (75.8, 93.6)
- added REF**: 2mmX3.5mmPadSMD, PCMCIA:2mmX3.5mmPadSMD, B.Cu at (94.5, 93.6)
- added REF**: 2mmX3.5mmPadSMD, PCMCIA:2mmX3.5mmPadSMD, B.Cu at (127.0, 93.6)
- added REF**: 2mmX3.5mmPadSMD, PCMCIA:2mmX3.5mmPadSMD, B.Cu at (77.3, 50.7)
- added REF**: 2mmX3.5mmPadSMD, PCMCIA:2mmX3.5mmPadSMD, B.Cu at (94.5, 50.7)
- added REF**: 2mmX3.5mmPadSMD, PCMCIA:2mmX3.5mmPadSMD, B.Cu at (124.2, 50.7)
Routing:
- net GND: track 350.8 -> 339.0 mm
- net /~OE: track 103.9 -> 102.4 mm
- net /D12: track 44.6 -> 43.4 mm
- net /D13: track 43.1 -> 42.0 mm
- net /D11: track 45.7 -> 44.7 mm
- net Vcc: track 209.8 -> 209.1 mm
- net /D15: track 40.2 -> 40.8 mm
- net /D14: track 42.2 -> 41.6 mm
Other:
- board size 78.5 x 47.2 mm -> 78.5 x 51.9 mm
- board text added: "I"
- board text added: "Write Enabled"
- board text added: "Write Protected"

Commit message: Updated FRAM Card PCB
Parts:
- removed the REF** at (115.8, 50.7)
- removed the REF** at (115.8, 93.6)
- removed the REF** at (75.8, 93.6)
- removed the REF** at (94.5, 93.6)
- removed the REF** at (127.0, 93.6)
- removed the REF** at (77.3, 50.7)
- removed the REF** at (94.5, 50.7)
- removed the REF** at (124.2, 50.7)
- added REF**: 2mmX3.5mmPadSMD, PCMCIA:2mmX3.5mmPadSMD, B.Cu at (74.4, 101.7)
- added REF**: 2mmX3.5mmPadSMD, PCMCIA:2mmX3.5mmPadSMD, B.Cu at (78.5, 101.8)
- added REF**: 2mmX3.5mmPadSMD, PCMCIA:2mmX3.5mmPadSMD, B.Cu at (132.5, 50.2)
- added REF**: 2mmX3.5mmPadSMD, PCMCIA:2mmX3.5mmPadSMD, B.Cu at (74.1, 50.2)
- added REF**: 2mmX3.5mmPadSMD, PCMCIA:2mmX3.5mmPadSMD, B.Cu at (121.3, 99.9)
- added REF**: 2mmX3.5mmPadSMD, PCMCIA:2mmX3.5mmPadSMD, B.Cu at (89.4, 52.1)
- added REF**: 2mmX3.5mmPadSMD, PCMCIA:2mmX3.5mmPadSMD, B.Cu at (93.1, 50.5)
- added REF**: 2mmX3.5mmPadSMD, PCMCIA:2mmX3.5mmPadSMD, B.Cu at (89.4, 99.9)
- added REF**: 2mmX3.5mmPadSMD, PCMCIA:2mmX3.5mmPadSMD, B.Cu at (121.0, 52.1)
- added REF**: 2mmX3.5mmPadSMD, PCMCIA:2mmX3.5mmPadSMD, B.Cu at (78.4, 50.1)
- added REF**: 2mmX3.5mmPadSMD, PCMCIA:2mmX3.5mmPadSMD, B.Cu at (128.5, 101.9)
- added REF**: 2mmX3.5mmPadSMD, PCMCIA:2mmX3.5mmPadSMD, B.Cu at (128.4, 50.1)
- moved R4 0.97 mm to (75.3, 58.9)
Connections:
- net /~BVD1 renamed /~{BVD1}
- net /~BVD2 renamed /~{BVD2}
- net /~CE1 renamed /~{CE1}
- net /~CE2 renamed /~{CE2}
- net /~OE renamed /~{OE}
- net /~REG renamed /~{REG}
- net /~VS1 renamed /~{VS1}
- net /~VS2 renamed /~{VS2}
- net /~WAIT renamed /~{WAIT}
- net /~WE renamed /~{WE}
- net /~WE~orWP renamed /~{WE}orWP
Routing:
- net GND: track 339.0 -> 344.7 mm
- net /A8: track 60.3 -> 57.7 mm
- net /A13: track 58.8 -> 56.5 mm
- net Vcc: track 209.1 -> 208.0 mm
- net Net-(D1-Pad2): track 16.6 -> 15.7 mm
- net Net-(D1-Pad1): track 26.9 -> 26.0 mm
- net /WP: track 88.4 -> 89.2 mm
- net /D9: track 89.3 -> 89.9 mm
- net /D8: track 89.9 -> 90.6 mm
- net /D10: track 89.3 -> 90.0 mm
Other:
- board size 78.5 x 51.9 mm -> 78.5 x 47.2 mm
- net class Default removed
- board text added: "FM TOWNS RESCUE BOOT MEMORY CARD Using HIROSE NX1 PCMCIA FRAME by Captain YS http://www.ysflight.com Ver. 20231127"
- board text removed: "FM TOWNS RESCUE BOOT MEMORY CARD Using HIROSE NX1 PCMCIA FRAME by Captain YS http://www.ysflight.com Ver. 20220525"

Commit message: Updated PCB
Other:
- board size 78.5 x 47.2 mm -> 79.6 x 47.2 mm
Changed lines of the file:
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@@
   (gr_line (start 75.33279 99.51359) (end 69.35 99.55)
     (stroke (width 0.05) (type solid)) (layer "Edge.Cuts"))
-  (gr_line (start 141.35 52.3748) (end 141.35 99.55)
+  (gr_line (start 142.3924 54.3052) (end 142.3924 97.6196)
     (stroke (width 0.05) (type solid)) (layer "Edge.Cuts"))
   (gr_line (start 75.33279 52.37841) (end 69.35 52.35)
@@
   (gr_line (start 141.35 99.55) (end 131.47401 99.56439)
     (stroke (width 0.05) (type solid)) (layer "Edge.Cuts"))
+  (gr_line (start 141.35 52.3748) (end 141.35 54.3052)
+    (stroke (width 0.05) (type default)) (layer "Edge.Cuts"))
   (gr_arc (start 120.28718 52.3748) (mid 120.64639 52.52359) (end 120.79518 52.8828)
     (stroke (width 0.05) (type default)) (layer "Edge.Cuts"))
@@
     (stroke (width 0.05) (type solid)) (layer "Edge.Cuts"))
   (gr_line (start 75.8444 97.9424) (end 75.84079 99.00559)
+    (stroke (width 0.05) (type default)) (layer "Edge.Cuts"))
+  (gr_line (start 141.35 54.3052) (end 142.3924 54.3052)
     (stroke (width 0.05) (type default)) (layer "Edge.Cuts"))
   (gr_arc (start 75.84079 99.00559) (mid 75.692 99.3648) (end 75.33279 99.51359)
@@
   (gr_arc (start 130.9624 52.8828) (mid 131.11119 52.52359) (end 131.4704 52.3748)
     (stroke (width 0.05) (type default)) (layer "Edge.Cuts"))
+  (gr_line (start 141.35 97.6196) (end 142.3924 97.6196)
+    (stroke (width 0.05) (type default)) (layer "Edge.Cuts"))
   (gr_arc (start 89.86881 52.88641) (mid 90.0176 52.5272) (end 90.37681 52.37841)
     (stroke (width 0.05) (type default)) (layer "Edge.Cuts"))
   (gr_line (start 129.93918 52.8828) (end 129.94279 53.94599)
     (stroke (width 0.05) (type default)) (layer "Edge.Cuts"))
+  (gr_line (start 141.35 97.6196) (end 141.35 99.55)
+    (stroke (width 0.05) (type default)) (layer "Edge.Cuts"))
   (gr_arc (start 88.33759 52.37841) (mid 88.6968 52.5272) (end 88.84559 52.88641)

Commit message: Updated FRAM card for NX case PCB.
Other:
- board text added: "FM TOWNS RESCUE BOOT MEMORY CARD Using HIROSE NX1 PCMCIA FRAME by Captain YS http://www.ysflight.com Ver. 20231206"
- board text removed: "FM TOWNS RESCUE BOOT MEMORY CARD Using HIROSE NX1 PCMCIA FRAME by Captain YS http://www.ysflight.com Ver. 20231127"
Changed lines of the file:
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@@
   (gr_line (start 120.79518 52.8828) (end 120.79879 53.94599)
     (stroke (width 0.05) (type default)) (layer "Edge.Cuts"))
-  (gr_text "FM TOWNS RESCUE BOOT MEMORY CARD\nUsing HIROSE NX1 PCMCIA FRAME\nby Captain YS  http://www.ysflight.com\nVer. 20231127" (at 123.825 66.548) (layer "B.SilkS")
+  (gr_text "FM TOWNS RESCUE BOOT MEMORY CARD\nUsing HIROSE NX1 PCMCIA FRAME\nby Captain YS  http://www.ysflight.com\nVer. 20231206" (at 123.825 66.548) (layer "B.SilkS")
     (effects (font (size 1.5 1.5) (thickness 0.3)) (justify left mirror))
   )
